File: esp8bit.kicad_pcb (KiCad board)
At the start: 2 copper layers, 85.9 x 50 mm, 10 parts, among them J1 Touchscreen, J2 Mini-DIN_6, J3 SD, J4 Sound, J5 Barrel_Jack_Switch, U1 WeMos_mini, U2 LM7805_TO220

Commit message: updates
Parts:
- added C3: 10u, Capacitor_THT:CP_Radial_D5.0mm_P2.00mm, F.Cu at (122.9, 86.0)
- added C4: 10u, Capacitor_THT:CP_Radial_D5.0mm_P2.00mm, F.Cu at (135.8, 65.4)
- added C5: 10u, Capacitor_THT:CP_Radial_D5.0mm_P2.00mm, F.Cu at (133.0, 86.1)
- added C6: 100n, Capacitor_THT:C_Disc_D6.0mm_W2.5mm_P5.00mm, F.Cu at (148.1, 66.8)
- added C7: 100u, Capacitor_THT:CP_Radial_D5.0mm_P2.00mm, F.Cu at (152.7, 86.1)
- added J6: Audio, Connector_PinHeader_2.54mm:PinHeader_1x03_P2.54mm_Horizontal, F.Cu at (145.3, 86.4)
- added R2: 100R, Resistor_THT:R_Axial_DIN0207_L6.3mm_D2.5mm_P10.16mm_Horizontal, F.Cu at (96.0, 80.5)
- added R3: 10k, Resistor_THT:R_Axial_DIN0207_L6.3mm_D2.5mm_P10.16mm_Horizontal, F.Cu at (141.5, 47.9)
- added R4: 27k, Resistor_THT:R_Axial_DIN0207_L6.3mm_D2.5mm_P10.16mm_Horizontal, F.Cu at (126.7, 71.5)
- added R5: 27k, Resistor_THT:R_Axial_DIN0207_L6.3mm_D2.5mm_P10.16mm_Horizontal, F.Cu at (116.6, 74.5)
- added R6: 10R, Resistor_THT:R_Axial_DIN0207_L6.3mm_D2.5mm_P10.16mm_Horizontal, F.Cu at (155.3, 80.3)
- added R7: 10k, Resistor_THT:R_Axial_DIN0207_L6.3mm_D2.5mm_P10.16mm_Horizontal, F.Cu at (151.6, 54.7)
- added R_POT1: 10k, Potentiometer_THT:Potentiometer_Bourns_3386P_Vertical, F.Cu at (113.7, 86.4)
- added U3: LM386, Package_DIP:DIP-8_W7.62mm_Socket, F.Cu at (140.7, 70.6)
- C1: value 220u -> 10n; footprint Capacitor_THT:CP_Radial_D6.3mm_P2.50mm -> Capacitor_THT:C_Disc_D6.0mm_W2.5mm_P5.00mm
- C2: value 22u -> 10n; footprint Capacitor_THT:CP_Radial_D5.0mm_P2.50mm -> Capacitor_THT:C_Disc_D6.0mm_W2.5mm_P5.00mm
- J1, J3: moved to F.Cu
- J2: value Mini-DIN_6 -> SD/RAM; footprint Custom_Footprints:Connector_Mini-DIN_Female_6Pin_2rows -> Connector_PinHeader_2.54mm:PinHeader_2x02_P2.54mm_Vertical
- J4: value Sound -> KBD; footprint Connector_PinHeader_2.54mm:PinHeader_1x03_P2.54mm_Vertical -> Connector_PinHeader_2.54mm:PinHeader_1x04_P2.54mm_Horizontal
- J5: value Barrel_Jack_Switch -> Backlight; footprint Connector_BarrelJack:BarrelJack_CUI_PJ-102AH_Horizontal -> Connector_PinHeader_2.54mm:PinHeader_2x02_P2.54mm_Vertical
- U2: value LM7805_TO220 -> 23K256-I_P; footprint Package_TO_SOT_THT:TO-220-3_Horizontal_TabDown -> Package_DIP:DIP-8_W7.62mm_Socket
- moved J5 69.3 mm to (85.3, 79.0), turned to 0 degrees
- moved J4 43.1 mm to (101.6, 86.4), turned to 270 degrees
- moved J1 32.9 mm to (78.7, 49.0)
- moved R1 32.6 mm to (118.2, 57.5), turned to 90 degrees
- moved C2 29.8 mm to (130.5, 74.6), turned to 0 degrees
- moved J2 27.6 mm to (117.0, 62.7), turned to 0 degrees
- moved U1 22.6 mm to (98.8, 56.9), turned to 180 degrees
- moved C1 19.5 mm to (130.5, 71.5), turned to 0 degrees
- moved U2 13.3 mm to (125.6, 47.9), turned to 0 degrees
- moved J3 7.62 mm to (160.5, 61.7)
Connections:
- C1 pad 1: +9V -> Net-(C1-Pad1)
- C2 pad 1: VCC -> Net-(C2-Pad1)
- J1 pad 8: VCC -> /LED
- J2 pad 1: /KBD_DATA -> /SD_RAM_CS
- J2 pad 2: Net-(J2-Pad2) -> /SD_CS
- J2 pad 3: GND -> /SD_RAM_CS
- J2 pad 4: VCC -> /RAM_CS
- J4 pad 1: GND -> /KBD_CLK
- J4 pad 2: /Sound -> /KBD_DATA
- J4 pad 3: VCC -> GND
- J5 pad 1: +9V -> /LED
- J5 pad 3: GND -> /LED
- R1 pad 1: /SD_CS -> /RAM_CS
- U1 pad 10: Net-(U1-Pad10) -> /A_IN
- U1 pad 11: /SD_CS -> /SD_RAM_CS
- U1 pad 16: Net-(U1-Pad16) -> +3V3
- U1 pad 3: /KBD_CLK -> /KBD_DATA
- U2 pad 1: +9V -> /RAM_CS
- U2 pad 2: GND -> /MISO
- U2 pad 3: VCC -> GND
Routing:
- net /A_IN: track 0.00 -> 61.9 mm
- net VCC: track 90.8 -> 150.6 mm
- net +3V3: track 0.00 -> 56.1 mm
- net GND: track 109.8 -> 154.9 mm
- net /Rst: track 56.9 -> 16.7 mm
- net /TFT_CS: track 46.8 -> 9.58 mm
- net /SD_RAM_CS: track 0.00 -> 32.9 mm
- net +9V: track 32.2 -> 0.00 mm
- net Net-(R_POT1-Pad2): track 0.00 -> 29.8 mm
- net Net-(C2-Pad1): track 0.00 -> 28.5 mm
- net /SD_CS: track 72.6 -> 47.2 mm
- net /RAM_CS: track 0.00 -> 21.4 mm
- net Net-(C5-Pad1): track 0.00 -> 20.9 mm
- net Net-(R3-Pad2): track 0.00 -> 19.5 mm
- net /Sound: track 32.5 -> 14.7 mm
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Other:
- board text added: "clk"
- board text added: "esp8bit v1.2 (c) 2021 steve"
- board text added: "in"
- board text added: "out"
- board text added: "pwm"
- board text added: "sd"
- board text added: "spiram"
- board text added: "vcc"
- board text removed: "esp8bit v1.0 (c) 2019 steve"
